File: pcb/mcu.kicad_sch (KiCad schematic)
At the start: 24 parts, among them J2 AVR-UPDI-UART-6, U4 ATtiny1616-MNR

Commit message: fixed extra spaces and sheet numbers
Parts:
- R13, R14: MN FOJAN -> FOJAN
